Commit message: update

File: universal_robot/ur_description/urdf/ur.xacro (robot description, xacro)
@@ -1,4 +1,4 @@
 <?xml version="1.0"?>
-<robot xmlns:xacro="http://wiki.ros.org/xacro" name="$(arg robot_model)_robot">
+<robot xmlns:xacro="http://wiki.ros.org/xacro" name="ur">
    <!-- import main macro -->
    <xacro:include filename="$(find ur_description)/urdf/inc/ur_macro.xacro"/>

File: universal_robot/ur_gazebo/urdf/ur.xacro (robot description, xacro)
@@ -1,4 +1,4 @@
 <?xml version="1.0"?>
-<robot xmlns:xacro="http://wiki.ros.org/xacro" name="$(arg robot_model)_robot">
+<robot xmlns:xacro="http://wiki.ros.org/xacro" name="ur_robot_gazebo">
   <!--
     This is a top-level xacro instantiating the Gazebo-specific version of the
@@ -38,5 +38,5 @@
           controller .yaml files in the 'config' directory.
   -->
-  <xacro:arg name="transmission_hw_interface" default="hardware_interface/EffortJointInterface"/>
+  <xacro:arg name="transmission_hw_interface" default="hardware_interface/PositionJointInterface"/>
   <xacro:arg name="safety_limits" default="false"/>
   <xacro:arg name="safety_pos_margin" default="0.15"/>
@@ -67,9 +67,3 @@
     <origin xyz="0 0 0" rpy="0 0 0"/>
   </joint>
-  <link name="tool0_controller"/>
-  <joint name="tool_controller_fake_joint" type="fixed">
-    <parent link="tool0"/>
-    <child link="tool0_controller"/>
-    <origin xyz="0 0 0" rpy="0 0 0"/>
-  </joint>
 </robot>

File: universal_robot/ur_gazebo/urdf/ur_macro.xacro (robot description, xacro)
@@ -37,5 +37,5 @@
    physical_parameters_file
    visual_parameters_file
-   transmission_hw_interface:=hardware_interface/EffortJointInterface
+   transmission_hw_interface:=hardware_interface/PositionJointInterface
    safety_limits:=false safety_pos_margin:=0.15 safety_k_position:=20"
   >
@@ -46,5 +46,5 @@
       the definitions for the real robot.
     -->
-  <xacro:include filename="$(find ur_description)/urdf/inc/ur_macro.xacro"/>
+    <xacro:include filename="$(find ur_description)/urdf/inc/ur_macro.xacro"/>
     <!-- Instantiate model for the REAL robot. -->
     <xacro:ur_robot
