Commit message: add camera model

File: dual_ur/dual_ur_description/urdf/robotiq_hande_gripper.urdf.xacro (robot description, xacro)
@@ -48,5 +48,5 @@
         <!-- Attach the robotiq hand-e gripper -->
         <xacro:robotiq_hande_gripper prefix="${prefix}" parent="${parent}">
-            <origin xyz="0 0 0.004" rpy="${pi/2.0} 0 ${pi/2}"/>
+            <origin xyz="0 0 0.004" rpy="0 0 0"/>
         </xacro:robotiq_hande_gripper>
         <!-- Gazebo FT sensor plugin -->

File: dual_ur/dual_ur_gazebo/urdf/dual_ur_gripper_hande.xacro (robot description, xacro)
@@ -42,5 +42,5 @@
         safety_pos_margin="$(arg safety_pos_margin)"
         safety_k_position="$(arg safety_k_position)"
-      >
+        >
         <origin xyz="0.0 +0.47 0.0" rpy="0.0 0.0 ${pi}" />
       </xacro:ur_gripper_hande>

File: dual_ur/dual_ur_gazebo/urdf/ur_gripper_hande.xacro (robot description, xacro)
@@ -33,4 +33,16 @@
     <xacro:include filename="$(find dual_ur_description)/urdf/robotiq_hande_gripper.urdf.xacro" />
     <xacro:robotiq_hande_gripper prefix="${prefix}" parent="${prefix}tool0" ft_prefix="${ft_prefix}"/>
+    <!-- DepthAI camera -->
+    <xacro:include filename="$(find dual_ur_description)/urdf/depthai_macro.urdf.xacro"/>
+    <xacro:depthai_camera camera_name   = "${prefix}oak"
+                          parent        = "${prefix}tool0"
+                          camera_model  = "OAK-D"
+                          base_frame    = "${prefix}oak_pippo"
+                          cam_pos_x     = "0.0017758721902284543"
+                          cam_pos_y     = "0.05171514529791572"
+                          cam_pos_z     = "0.10236570223276018"
+                          cam_roll      = "0.0"
+                          cam_pitch     = "0.0"
+                          cam_yaw       = "0.0" />
   </xacro:macro>
 </robot>
