Commit message: camera model changed

File: dual_ur/dual_ur_description/urdf/depthai_macro.urdf.xacro (robot description, xacro)
@@ -4,13 +4,8 @@
                                            cam_pos_x cam_pos_y cam_pos_z
                                            cam_roll cam_pitch cam_yaw
-                                           r:=0.8 g:=0.8 b:=0.8 a:=0.8">
-    <xacro:property name="M_PI"     value="3.1415926535897931" />
-    <xacro:property name="model"    value="${camera_model}" />
+                                           r:=0.6 g:=0.6 b:=0.6 a:=1.0">
     <xacro:property name="has_imu" value="false" />
-    <!-- <xacro:if value="${model == 'BW1098OAK'}">
-    </xacro:if> -->
     <xacro:property name="baseline" value="0.075" />
-    <xacro:if value="${model == 'OAK-D'}">
-      <xacro:property name="has_imu" value="true" />
+    <xacro:if value="${camera_model == 'OAK-D'}">
       <xacro:property name="imu_offset_x" value="0.0" />
       <xacro:property name="imu_offset_y" value="-0.015" />
@@ -27,10 +22,10 @@
         <origin xyz="${cam_pos_x} ${cam_pos_y} ${cam_pos_z}" rpy="${cam_roll} ${cam_pitch} ${cam_yaw}" />
     </joint>
-<!-- device Center -->
+    <!-- device Center -->
     <link name="${camera_name}_model_origin">
         <visual>
-            <origin xyz="0 0 0" rpy="0.0 ${M_PI/2} ${M_PI/2}"/>
+            <origin xyz="0 0 0" rpy="0.0 ${pi/2} ${pi/2}"/>
             <geometry>
-                <mesh filename="package://dual_ur_description/model/camera_model/${model}.stl" />
+                <mesh filename="package://dual_ur_description/model/camera_model/${camera_model}.stl" />
             </geometry>
             <material name="mat">
@@ -39,12 +34,13 @@
         </visual>
         <collision>
-            <origin xyz="0 0 0" rpy="0.0 ${M_PI/2} ${M_PI/2}"/>
+            <origin xyz="0 0 0" rpy="0.0 ${pi/2} ${pi/2}"/>
             <geometry>
-                <mesh filename="package://dual_ur_description/model/camera_model/${model}.stl" />
+                <mesh filename="package://dual_ur_description/model/camera_model/${camera_model}.stl" />
             </geometry>
         </collision>
     </link>
     <joint name="${camera_name}_model_origin_joint" type="fixed">
-        <parent link="${base_frame}"/><!-- Left Camera -->
+        <parent link="${base_frame}"/>
+    <!-- Left Camera -->
     <link name="${camera_name}_left_camera_frame" />
     <joint name="${camera_name}_left_camera_joint" type="fixed">
@@ -55,9 +51,9 @@
     <link name="${camera_name}_left_camera_optical_frame"/>
     <joint name="${camera_name}_left_camera_optical_joint" type="fixed">
-        <origin xyz="0 0 0" rpy="-${M_PI/2} 0.0 -${M_PI/2}"/>
+        <origin xyz="0 0 0" rpy="-${pi/2} 0.0 -${pi/2}"/>
         <parent link="${camera_name}_left_camera_frame"/>
         <child link="${camera_name}_left_camera_optical_frame"/>
     </joint>
-<!-- right Camera -->
+    <!-- right Camera -->
     <link name="${camera_name}_right_camera_frame" />
     <joint name="${camera_name}_right_camera_joint" type="fixed">
@@ -68,5 +64,5 @@
     <link name="${camera_name}_right_camera_optical_frame"/>
     <joint name="${camera_name}_right_camera_optical_joint" type="fixed">
-        <origin xyz="0 0 0" rpy="-${M_PI/2} 0.0 -${M_PI/2}"/>
+        <origin xyz="0 0 0" rpy="-${pi/2} 0.0 -${pi/2}"/>
         <parent link="${camera_name}_right_camera_frame"/>
         <child link="${camera_name}_right_camera_optical_frame"/>
@@ -75,5 +71,5 @@
         <origin xyz="0 0 0" rpy="1.5708 0 1.5708" />
     </joint>
-<!-- IMU -->
+    <!-- IMU -->
     <xacro:if value="${has_imu}">
         <link name="${camera_name}_imu_frame" />
@@ -84,5 +80,5 @@
         </joint>
     </xacro:if>
-<!-- RGB Camera -->
+    <!-- RGB Camera -->
     <link name="${camera_name}_rgb_camera_frame" />
     <joint name="${camera_name}_rgb_camera_joint" type="fixed">
@@ -97,5 +93,6 @@
         <child link="${camera_name}_rgb_camera_optical_frame"/>
     </joint>
-<!-- Left Camera -->
+    <!-- Left Camera -->
+    <!--
     <link name="${camera_name}_left_camera_frame" />
     <joint name="${camera_name}_left_camera_joint" type="fixed">
@@ -106,9 +103,11 @@
     <link name="${camera_name}_left_camera_optical_frame"/>
     <joint name="${camera_name}_left_camera_optical_joint" type="fixed">
-        <origin xyz="0 0 0" rpy="-${M_PI/2} 0.0 -${M_PI/2}"/>
+        <origin xyz="0 0 0" rpy="-${pi/2} 0.0 -${pi/2}"/>
         <parent link="${camera_name}_left_camera_frame"/>
         <child link="${camera_name}_left_camera_optical_frame"/>
     </joint>
-<!-- right Camera -->
+    -->
+    <!-- right Camera -->
+    <!--
     <link name="${camera_name}_right_camera_frame" />
     <joint name="${camera_name}_right_camera_joint" type="fixed">
@@ -119,8 +118,9 @@
     <link name="${camera_name}_right_camera_optical_frame"/>
     <joint name="${camera_name}_right_camera_optical_joint" type="fixed">
-        <origin xyz="0 0 0" rpy="-${M_PI/2} 0.0 -${M_PI/2}"/>
+        <origin xyz="0 0 0" rpy="-${pi/2} 0.0 -${pi/2}"/>
         <parent link="${camera_name}_right_camera_frame"/>
         <child link="${camera_name}_right_camera_optical_frame"/>
     </joint>
+    -->
 </xacro:macro>
 </robot>
