Commit message: change urdf name

File: dual_ur/dual_ur_gazebo/urdf/dual_ur_gripper_hande.xacro (robot description, xacro)
@@ -1,4 +1,4 @@
 <?xml version="1.0"?>
-<robot xmlns:xacro="http://wiki.ros.org/xacro" name="ur_robot_gazebo">
+<robot xmlns:xacro="http://wiki.ros.org/xacro" name="dual_ur">
   <xacro:include filename="$(find dual_ur_gazebo)/urdf/ur_gripper_hande.xacro"/>
   <!--Declare arguments -->

File: dual_ur/dual_ur_gazebo/urdf/ur_gripper_hande.xacro (robot description, xacro)
@@ -1,4 +1,4 @@
 <?xml version="1.0"?>
-<robot xmlns:xacro="http://wiki.ros.org/xacro" name="ur_robot_gazebo">
+<robot xmlns:xacro="http://wiki.ros.org/xacro" name="dual_ur">
   <xacro:macro name="ur_gripper_hande" params="
     prefix
@@ -14,5 +14,5 @@
   <xacro:include filename="$(find dual_ur_gazebo)/urdf/ur_macro.xacro"/>
     <!-- Instantiate the Gazebo robot and pass it all the required arguments. -->
-    <xacro:ur_robot_gazebo
+    <xacro:dual_ur
       prefix="${prefix}"
       joint_limits_parameters_file="${joint_limits_parameters_file}"

File: dual_ur/dual_ur_gazebo/urdf/ur_macro.xacro (robot description, xacro)
@@ -31,5 +31,5 @@
   -->
   <!-- Definition of the main macro -->
-  <xacro:macro name="ur_robot_gazebo" params="
+  <xacro:macro name="dual_ur" params="
    prefix
    joint_limits_parameters_file
